Commit message: Add labo version

File: trooper_description/urdf/trooper_labo.urdf (robot description, URDF)
Before this commit: robot trooper, 7 links, 6 joints
Links:
- link trooper__chassis: geometry collision mesh filename=package://trooper_description/meshes/stl/chassis_no_guardra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 scale=0.01 0.01 0.01; visual mesh filename=package://trooper_description/meshes/stl/chassis_no_guardra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 scale=0.01 0.01 0.01
