Commit message: ADD: 4 layers lidar feature (first commit)

File: trooper_description/urdf/trooper.urdf.xacro (robot description, xacro)
@@ -1,5 +1,9 @@
 <?xml version="1.0"?>
 <robot name="trooper" xmlns:xacro="http://ros.org/wiki/xacro">
-<xacro:include filename="$(find velodyne_description)/urdf/VLP-16.urdf.xacro"/>
+	<xacro:property name="M_PI" value="3.1415926535897931" />
+	<xacro:arg name="gpu" default="false"/>
+	<xacro:property name="gpu" value="$(arg gpu)" />
+ 	<xacro:arg name="organize_cloud" default="true"/>
+ 	<xacro:property name="organize_cloud" value="$(arg organize_cloud)" />
 <!-- Color materials (Compatible with Rviz but not yet with Gazebo) -->
 	<material name="greenish">
@@ -138,4 +142,5 @@
 	</gazebo>
 <!-- SENSORS -->
+<!--
 	<link name="lidar">
 		<collision>
@@ -157,4 +162,5 @@
 		</inertial>
 	</link>
+	-->
 <link name="imu_link">
   <inertial>
@@ -212,4 +218,11 @@
     <!--<limit effort="10" velocity="100"/>-->
   </joint>
+	<joint name="imu_joint" type="fixed">
+		<axis xyz="1 0 0"/> <!-- 0 1 0 -->
+		<origin xyz="0 0 0.19"/>
+		<parent link="base_link"/>
+		<child link="imu_link"/>
+	</joint>
+<!--
   <property name="lidar" value="0.15" />
   <joint name="lidar_joint" type="fixed">
@@ -219,20 +232,16 @@
     <child link="lidar"/>
   </joint>
-	<VLP-16 parent="lidar" name="velodyne" topic="/cloud" hz="10" samples="440">
-		<origin xyz="0 0 °" rpy="0 0 0"/>
-		<samples>653</samples>
-		<lasers>4</lasers>
-		<min_angle>-1.3955</min_angle>
-		<max_angle>1.3955</max_angle>
-		<min_range>0.10</min_range>
-		<max_range>5.0</max_range>
-		<hz>10</hz>
-		 </VLP-16>
-  <joint name="imu_joint" type="fixed">
-    <axis xyz="1 0 0"/> <!-- 0 1 0 -->
-    <origin xyz="0 0 0.19"/>
-    <parent link="base_link"/>
-    <child link="imu_link"/>
-  </joint>
+-->
+<!--
+	<xacro:include filename="$(find velodyne_description)/urdf/VLP-16.urdf.xacro"/>
+	<xacro:VLP-16 parent="lidar" name="velodyne" topic="/cloud" organize_cloud="${organize_cloud}" hz="10" samples="653" gpu="${gpu}" lasers="4" min_angle="-1.3955"
+		max_angle="1.3955" min_range="0.10" max_range="5.0">
+	<origin xyz="0.04 0 0" rpy="0 0 0" />
+	</xacro:VLP-16>
+-->
+	<xacro:include filename="$(find velodyne_description)/urdf/VLP-16.urdf.xacro"/>
+  <xacro:VLP-16 parent="base_link" name="lidar" topic="/cloud" organize_cloud="${organize_cloud}" hz="10" samples="653" gpu="${gpu}">
+    <origin xyz="0.28 0 0.08" rpy="0 0 0"/>
+  </xacro:VLP-16>
 <!--  GAZEBO plugin for Laser -->
 <!--
@@ -263,11 +272,10 @@
         </range>
         <noise>
-          <type>gaussian</type>
-					-->
+          <type>gaussian</type>-->
           <!-- Noise parameters based on published spec for Hokuyo laser
                achieving "+-30mm" accuracy at range < 10m.  A mean of 0.0m and
                stddev of 0.01m will put 99.7% of samples within 0.03m of the true
                reading. -->
-							 <!--
+							   <!--
           <mean>0.0</mean>
           <stddev>0.01</stddev>
@@ -279,6 +287,5 @@
       </plugin>
     </sensor>
-  </gazebo>
--->
+  </gazebo>-->
 <!--  GAZEBO plugin for IMU -->
   <gazebo reference="imu_link">
@@ -328,5 +335,5 @@
     </actuator>
     <joint name="trooper__magasin_to_chassis">
-      <hardwareInterface>PositionJointInterface</hardwareInterface>
+      <hardwareInterface>hardware_interface/PositionJointInterface</hardwareInterface>
     </joint>
   </transmission>
@@ -337,5 +344,5 @@
     </actuator>
     <joint name="trooper__left_wheel_to_chassis">
-      <hardwareInterface>VelocityJointInterface</hardwareInterface>
+      <hardwareInterface>hardware_interface/VelocityJointInterface</hardwareInterface>
     </joint>
   </transmission>
@@ -346,5 +353,5 @@
     </actuator>
     <joint name="trooper__right_wheel_to_chassis">
-      <hardwareInterface>VelocityJointInterface</hardwareInterface>
+      <hardwareInterface>hardware_interface/VelocityJointInterface</hardwareInterface>
     </joint>
   </transmission>

Commit message: MOD: configuration du lidar dans l'urdf.xacro

File: trooper_description/urdf/trooper.urdf.xacro (robot description, xacro)
@@ -142,25 +142,4 @@
 	</gazebo>
 <!-- SENSORS -->
-<!--
-	<link name="lidar">
-		<collision>
-		  <origin xyz="0 0 0" rpy="0 0 0"/>
-		  <geometry>
-		    <box size="0.05 0.05 0.041"/>
-		  </geometry>
-		</collision>
-		<visual>
-		  <origin xyz="0 0 0" rpy="0 0 0"/>
-		  <geometry>
-		    <cylinder length="0.029" radius="0.021"/>
-		  </geometry>
-		</visual>
-		<inertial>
-		  <mass value="0.1" />
-		  <origin xyz="0 0 0" rpy="0 0 0"/>
-		  <inertia ixx="1" ixy="0" ixz="0" iyy="1" iyz="0" izz="1" />
-		</inertial>
-	</link>
-	-->
 <link name="imu_link">
   <inertial>
@@ -224,68 +203,9 @@
 		<child link="imu_link"/>
 	</joint>
-<!--
-  <property name="lidar" value="0.15" />
-  <joint name="lidar_joint" type="fixed">
-    <axis xyz="0 1 0" />
-    <origin xyz="0.28 0 0.08" rpy="0 0 0"/>
-    <parent link="base_link"/>
-    <child link="lidar"/>
-  </joint>
--->
-<!--
 	<xacro:include filename="$(find velodyne_description)/urdf/VLP-16.urdf.xacro"/>
-	<xacro:VLP-16 parent="lidar" name="velodyne" topic="/cloud" organize_cloud="${organize_cloud}" hz="10" samples="653" gpu="${gpu}" lasers="4" min_angle="-1.3955"
-		max_angle="1.3955" min_range="0.10" max_range="5.0">
-	<origin xyz="0.04 0 0" rpy="0 0 0" />
-	</xacro:VLP-16>
--->
-	<xacro:include filename="$(find velodyne_description)/urdf/VLP-16.urdf.xacro"/>
-  <xacro:VLP-16 parent="base_link" name="lidar" topic="/cloud" organize_cloud="${organize_cloud}" hz="10" samples="653" gpu="${gpu}">
+  <xacro:VLP-16 parent="base_link" name="lidar" topic="/cloud" organize_cloud="${organize_cloud}" hz="10" samples="653" gpu="${gpu}" lasers="4"
+		min_angle="-1.3955" max_angle="1.3955" min_range="0.1" max_range="5.0" >
     <origin xyz="0.28 0 0.08" rpy="0 0 0"/>
   </xacro:VLP-16>
-<!--  GAZEBO plugin for Laser -->
-<!--
-  <gazebo reference="lidar">
-    <sensor type="ray" name="head_hokuyo_sensor">
-      <pose>0 0 0 0 0 0</pose>
-      <visualize>true</visualize>
-      <update_rate>20</update_rate>
-      <ray>
-        <scan>
-          <horizontal>
-            <samples>653</samples>
-            <resolution>1</resolution>
-            <min_angle>-1.3955</min_angle>
-            <max_angle>1.3955</max_angle>
-          </horizontal>
-					<vertical>
-            <samples>4</samples>
-            <min_angle>-0.065</min_angle>
-            <max_angle>0.065</max_angle>
-            <resolution>1</resolution>
-          </vertical>
-        </scan>
-        <range>
-          <min>0.10</min>
-          <max>5.0</max>
-          <resolution>0.01</resolution>
-        </range>
-        <noise>
-          <type>gaussian</type>-->
-          <!-- Noise parameters based on published spec for Hokuyo laser
-               achieving "+-30mm" accuracy at range < 10m.  A mean of 0.0m and
-               stddev of 0.01m will put 99.7% of samples within 0.03m of the true
-               reading. -->
-							   <!--
-          <mean>0.0</mean>
-          <stddev>0.01</stddev>
-        </noise>
-      </ray>
-      <plugin name="velodyne_gazebo_plugins" filename="libgazebo_ros_laser.so">
-        <topicName>/scan</topicName>
-        <frameName>lidar</frameName>
-      </plugin>
-    </sensor>
-  </gazebo>-->
 <!--  GAZEBO plugin for IMU -->
   <gazebo reference="imu_link">
