Commit message: Split structure in 2 main directories: trooper_description (robot independent from environment) and trooper_gazebo (3d simulator independent from robot)

File: trooper_description/urdf/trooper.urdf (robot description, URDF)
Before this commit: robot trooper, 6 links, 5 joints
Links:
- removed link trooper__hokuyo__link
- added link hokuyo_link, mass 0.1; collision box size=0.05 0.05 0.041; visual cylinder length=0.029 radius=0.021
- link trooper__chassis: geometry collision mesh filename=package://trooper_description/meshes/stl/chassis.stl scale=0.01 0.01 0.01; visual mesh filename=package://trooper_description/meshes/stl/chassis.stl scale=0.01 0.01 0.01
- link trooper__left_wheel: geometry collision cylinder length=0.1 radius=0.15; visual mesh filename=package://trooper_description/meshes/stl/drive_wheel.stl scale=0.01 0.01 0.01
- link trooper__platform: geometry collision mesh filename=package://trooper_description/meshes/stl/platform_5x4L.stl scale=0.01 0.01 0.01; visual mesh filename=package://trooper_description/meshes/stl/platform_5x4L.stl scale=0.01 0.01 0.01
- link trooper__right_wheel: geometry collision cylinder length=0.1 radius=0.15; visual mesh filename=package://trooper_description/meshes/stl/drive_wheel.stl scale=0.01 0.01 0.01
Joints:
- removed joint trooper__hokuyo_joint
- added joint hokuyo_joint: type fixed, parent trooper__chassis, child hokuyo_link, origin xyz=0.28 0 0.08 rpy=0 0 0, axis 0 1 0

Commit message: trooper_chassis to base_link

File: trooper_description/urdf/trooper.urdf (robot description, URDF)
Before this commit: robot trooper, 7 links, 6 joints
Links:
- removed link trooper__chassis
- added link base_link, mass 40; collision mesh filename=package://trooper_description/meshes/stl/chassis.stl scale=0.01 0.01 0.01; visual mesh filename=package://trooper_description/meshes/stl/chassis.stl scale=0.01 0.01 0.01
Joints:
- joint hokuyo_joint: parent trooper__chassis -> base_link
- joint imu_joint: parent trooper__chassis -> base_link
- joint trooper__left_wheel_to_chassis: parent trooper__chassis -> base_link
- joint trooper__magasin_to_chassis: parent trooper__chassis -> base_link
- joint trooper__right_wheel_to_chassis: parent trooper__chassis -> base_link
- joint trooper__rim_to_chassis: parent trooper__chassis -> base_link
